Commit message: modify urdf and add  collision

File: aubo_description/urdf/aubo_i3.urdf (robot description, URDF)
Before this commit: robot aubo_i3, 8 links, 7 joints
Links:
- added link camera_link; visual box size=0.005 0.005 0.005
- added link ee_link; visual box size=0.005 0.005 0.005
- added link eef_link; collision mesh filename=package://aubo_description/meshes/aubo_i3/collision/eef_new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; visual mesh filename=package://aubo_description/meshes/aubo_i3/collision/eef_new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
- added link finger; visual box size=0.005 0.005 0.005
- added link mounter; collision mesh filename=package://aubo_description/meshes/aubo_i3/collision/mounter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; visual mesh filename=package://aubo_description/meshes/aubo_i3/collision/mounter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
- added link palm; visual box size=0.005 0.005 0.005
- added link tool0
Joints:
- added joint ee_fixed_joint: type fixed, parent wrist3_Link, child ee_link, origin xyz=0.0 0.0 0.0 rpy=0.0 0.0 1.57079
- added joint eef_joint: type fixed, parent ee_link, child eef_link, origin xyz=0.0 0.0 0.0 rpy=3.14159 -1.5708 0.0
- added joint eelink_finger_joint: type fixed, parent ee_link, child finger, origin xyz=0.181500 -0.071350 0.028340 rpy=0.59341 0 0
- added joint eelink_palm_joint: type fixed, parent ee_link, child palm, origin xyz=0.188930 0.005870 0.059050 rpy=0.59341 0 0
- added joint mounter_joint: type fixed, parent mounter, child base_link, origin xyz=0.0 0 0.0 rpy=3.14159 0.0 5.49780
- added joint vision_joint: type fixed, parent ee_link, child camera_link, origin xyz=-0.172481 0.102860 -0.090900 rpy=0.105282 -0.048103 -0.107558
- added joint wrist3_Link-tool0_fixed_joint: type fixed, parent wrist3_Link, child tool0, origin xyz=0 0 0 rpy=-1.57079 0 0
- joint foreArm_joint: limit lower=-3.05 upper=3.05 effort=0 velocity=0 -> lower=-2.96705 upper=-0.08726 effort=0 velocity=0
- joint shoulder_joint: limit lower=-3.05 upper=3.05 effort=0 velocity=0 -> lower=-5.41052 upper=1.74532 effort=0 velocity=0
- joint upperArm_joint: limit lower=-3.05 upper=3.05 effort=0 velocity=0 -> lower=-3.31612 upper=-0.78539 effort=0 velocity=0
- joint world_joint: child base_link -> mounter; origin xyz=0.0 0.0 0.0 rpy=0.0 0.0 0.0 -> xyz=0.0 -0.658 0.0 rpy=0 0 0.02618
- joint wrist1_joint: limit lower=-3.05 upper=3.05 effort=0 velocity=0 -> lower=-4.71239 upper=0.0 effort=0 velocity=0
- joint wrist2_joint: limit lower=-3.05 upper=3.05 effort=0 velocity=0 -> lower=-1.57080 upper=0.0 effort=0 velocity=0
- joint wrist3_joint: limit lower=-3.05 upper=3.05 effort=0 velocity=0 -> lower=-1.29154 upper=2.96705 effort=0 velocity=0

Commit message: test

File: aubo_description/urdf/aubo_i3.urdf (robot description, URDF)
Before this commit: robot aubo_i3, 15 links, 14 joints
Links:
- link eef_link: mass None -> 0.1
- link mounter: mass None -> 0.1

File: aubo_description/urdf/aubo_i3.urdf.xacro (robot description, xacro)
@@ -206,7 +206,31 @@
   <link name="world" />
   <joint name="world_joint" type="fixed">
-    <parent link="world" />
-    <child link = "base_link" />
-    <origin xyz="0.0 0.0 0.0" rpy="0.0 0.0 0.0" />
+    <parent link="world"/>
+    <child link="mounter"/>
+    <origin xyz="0.0 -0.658 0.0" rpy="0 0 0"/>
+  </joint>
+  <link name="mounter">
+    <visual>
+      <geometry>
+        <mesh filename="package://aubo_description/meshes/aubo_i3/collision/mounter_front_new.stl"/>
+      </geometry>
+      <material name="LightGrey">
+        <color rgba="0.7 0.7 0.7 1.0"/>
+      </material>
+    </visual>
+    <collision>
+      <geometry>
+        <mesh filename="package://aubo_description/meshes/aubo_i3/collision/mounter_front_new.stl"/>
+      </geometry>
+    </collision>
+    <inertial>
+      <mass value="0.1"/>
+      <inertia ixx="0.00003" iyy="0.00003" izz="0.00003" ixy="0.0" ixz="0.0" iyz="0.0"/>
+    </inertial>
+  </link>
+  <joint name="mounter_joint" type="fixed">
+    <parent link="mounter"/>
+    <child link="base_link"/>
+    <origin xyz="0.0 0 0.0" rpy="3.14159 0.0 5.49780"/>
   </joint>
 </robot>

Commit message: test

File: aubo_description/urdf/aubo_i3.urdf (robot description, URDF)
Before this commit: robot aubo_i3, 15 links, 14 joints
Joints:
- joint ee_fixed_joint: origin xyz=0.0 0.0 0.0 rpy=0.0 0.0 1.57079 -> xyz=0.0 0.0 0.0 rpy=0.0 -1.57079 0
- joint eef_joint: origin xyz=0.0 0.0 0.0 rpy=3.14159 -1.5708 0.0 -> xyz=0.0 0.0 0.0 rpy=0 0 0.0
